File: kicad/ESP32_BNO086/ESP32_BNO086.kicad_pcb (KiCad board)
At the start: 2 copper layers, 35.9 x 20 mm, 14 parts, among them IC1 BNO086, U1 XIAO-ESP32-C3/S3

Commit message: wiring changes
Parts:
- removed RST/Center1: SW_Push, Button_Switch_SMD:SW_SPST_EVQP2_MiddlePushTravel_H2.5mm
- added C4: 0.1uf, Capacitor_SMD:C_0402_1005Metric, B.Cu at (138.9, 88.8)
- C3: value 0.1uf -> 10uf
- moved FUNC1 11.0 mm to (162.4, 87.3)
- moved LS1 4.03 mm to (162.4, 96.7)
- moved C3 1.11 mm to (138.9, 87.9), turned to 180 degrees
- moved R2 0.70 mm to (157.1, 88.2)
- moved R1 0.70 mm to (158.6, 88.2)
Connections:
- C3 pad 1: Net-(IC1-PS0/WAKE) -> Net-(IC1-PS1)
- C3 pad 2: Net-(IC1-VDD) -> GND
- FUNC1 pad 2: Net-(U1-GPIO21_D6_TX) -> Net-(U1-GPIO7_D5_SCL)
- IC1 pad 28: unconnected-(IC1-VDDIO-Pad28) -> Net-(IC1-PS1)
- IC1 pad 3: Net-(IC1-VDD) -> Net-(IC1-PS1)
- IC1 pad 5: Net-(IC1-PS0/WAKE) -> Net-(IC1-PS1)
- LS1 pad LOAD+: Net-(U1-GPIO7_D5_SCL) -> Net-(U1-GPIO21_D6_TX)
- PH2.0 pad MP: GND -> (no net)
- U1 pad 12: Net-(IC1-PS0/WAKE) -> Net-(IC1-PS1)
- U1 pad 3: Net-(IC1-H_CSN) -> Net-(IC1-PS0/WAKE)
- U1 pad 4: Net-(IC1-H_INTN) -> Net-(IC1-H_CSN)
- U1 pad 5: Net-(U1-GPIO6_D4_SDA) -> Net-(IC1-H_INTN)
Routing:
- net Net-(U1-GPIO6_D4_SDA): track 20.6 -> 0.00 mm
- net Net-(IC1-PS1): track 0.00 -> 17.5 mm, vias 0 -> 2
- net Net-(IC1-PS0/WAKE): track 9.82 -> 14.5 mm, vias 0 -> 2
- net Net-(U1-GPIO7_D5_SCL): track 14.5 -> 19.2 mm
- net Net-(IC1-VDD): track 4.66 -> 0.00 mm
- net Net-(IC1-H_CSN): track 14.6 -> 12.4 mm
- net Net-(U1-GPIO21_D6_TX): track 9.32 -> 10.3 mm

Commit message: Updated PCB design
Parts:
- added C5: 100nf, Capacitor_SMD:C_0402_1005Metric, B.Cu at (142.5, 89.5)
- added R4: 10k, Resistor_SMD:R_0402_1005Metric, B.Cu at (139.2, 92.4)
- moved C4 0.65 mm to (138.2, 88.8)
- moved C3 0.65 mm to (138.2, 87.9)
Connections:
- IC1 pad 4: unconnected-(IC1-BOOTN-Pad4) -> Net-(IC1-BOOTN)
- IC1 pad 9: unconnected-(IC1-CAP-Pad9) -> Net-(IC1-CAP)
Routing:
- net Net-(IC1-PS1): track 17.5 -> 19.5 mm
- net Net-(IC1-BOOTN): track 0.00 -> 1.07 mm
- net Net-(IC1-CAP): track 0.00 -> 1.01 mm
- net GND: vias 8 -> 10
Other:
- board size 35.9 x 20 mm -> 35.9 x 20.1 mm
- board text added: "+"
- board text added: "-"

Commit message: PCB tweaks again
Routing:
- net GND: track 3.85 -> 3.66 mm, vias 10 -> 9
- net /Bat+: vias 1 -> 0
Changed lines of the file:
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@@
-	)
-	(segment
-		(start 140.902 97.102)
-		(end 140.929 97.075)
-		(width 0.2)
-		(layer "F.Cu")
-		(net 13)
-	)
-	(segment
-		(start 140.804 97.2)
-		(end 140.902 97.102)
-		(width 0.2)
-		(layer "F.Cu")
-		(net 13)
 	)
 	(segment
@@
 		(layers "F.Cu" "B.Cu")
 		(free yes)
-		(net 13)
-	)
-	(via
-		(at 140.902 97.102)
-		(size 1)
-		(drill 0.5)
-		(layers "F.Cu" "B.Cu")
 		(net 13)
 	)
@@
 	)
 	(segment
-		(start 140.902 97.102)
-		(end 140.892 97.102)
-		(width 0.2)
-		(layer "B.Cu")
-		(net 13)
-	)
-	(segment
 		(start 143.22 85.01)
 		(end 146.7 88.49)
@@
 		(net 26)
 	)
-	(via
-		(at 142.834 97.075)
-		(size 1)
-		(drill 0.5)
-		(layers "F.Cu" "B.Cu")
-		(net 26)
-	)
