File: kicad/ESP32_BNO086/ESP32_BNO086.kicad_pcb (KiCad board)
At the start: 2 copper layers, 35.9 x 20.1 mm, 16 parts, among them IC1 BNO086, U1 XIAO-ESP32-C3/S3

Commit message: pcb updates, doc updates, lib updates
Parts:
- removed LS1: SMT-0540-T-9-R, 1_MyFootPrints:XDCR_SMT-0540-T-9-R
- removed S1: JS102011SAQN, 1_MyFootPrints:SW_JS102011SAQN
- added BUZZER1: MLT-5020, 1_MyFootPrints:BUZ-SMD_L5.0-W5.5-P4.60, B.Cu at (162.4, 96.9)
- added PWR1: K3-1280S-K1, 1_MyFootPrints:SW-SMD_K3-1280S-K1, F.Cu at (163.2, 87.7)
- added R5: 10k, Resistor_SMD:R_0402_1005Metric, B.Cu at (140.4, 89.0)
- added R6: 10k, Resistor_SMD:R_0402_1005Metric, B.Cu at (143.0, 88.6)
- added R7: 4.7k, Resistor_SMD:R_0402_1005Metric, B.Cu at (145.5, 89.4)
- added R8: 4.7k, Resistor_SMD:R_0402_1005Metric, B.Cu at (146.5, 89.4)
- C3, C4: footprint Capacitor_SMD:C_0402_1005Metric -> Capacitor_SMD:C_0603_1608Metric
- FUNC1: value SW_Push -> HX 3X4X2-2P-1.6N TACTILE SWITCH; footprint Button_Switch_SMD:SW_SPST_EVQP2_MiddlePushTravel_H2.5mm -> 1_MyFootPrints:KEY-SMD_L4.0-W3.0-LS4.9-1
- PH2.0: value Conn_01x02_Socket -> S2B-PH-SM4-TB(LF)(SN)
- U1: value XIAO-ESP32-C3/S3 -> XIAO-ESP32-C3
- moved R1 4.49 mm to (156.6, 84.1), turned to 0 degrees
- moved PH2.0 4.24 mm to (158.6, 98.0), turned to 90 degrees
- moved R2 2.57 mm to (156.6, 85.6), turned to 0 degrees
- moved C3 2.33 mm to (138.0, 90.2), turned to 0 degrees
- moved C1 1.83 mm to (160.4, 84.9)
- moved C2 1.83 mm to (158.9, 84.9)
- moved C5 1.11 mm to (141.8, 88.6)
- moved FUNC1 0.58 mm to (162.4, 87.9), turned to 90 degrees
- moved C4 0.33 mm to (138.0, 88.7), turned to 0 degrees
Connections:
- C3 pad 1: Net-(IC1-PS1) -> GND
- C3 pad 2: GND -> Net-(IC1-PS1)
- C4 pad 1: Net-(IC1-PS1) -> GND
- C4 pad 2: GND -> Net-(IC1-PS1)
- FUNC1 pad 1: GND -> Net-(U1-GPIO7_D5_SCL)
- FUNC1 pad 2: Net-(U1-GPIO7_D5_SCL) -> GND
- IC1 pad 10: unconnected-(IC1-CLKSEL0-Pad10) -> Net-(IC1-CLKSEL0)
- IC1 pad 15: unconnected-(IC1-ENV_SCL-Pad15) -> Net-(IC1-ENV_SCL)
- IC1 pad 16: unconnected-(IC1-ENV_SDA-Pad16) -> Net-(IC1-ENV_SDA)
Routing:
- net Net-(IC1-PS1): track 19.5 -> 29.4 mm, vias 2 -> 4
- net /Bat+: track 40.3 -> 47.1 mm
- net Net-(U1-GPIO7_D5_SCL): track 19.2 -> 23.0 mm
- net Net-(IC1-ENV_SDA): track 0.00 -> 2.36 mm
- net Net-(U1-GPIO2_A0_D0): track 27.6 -> 29.8 mm, vias 0 -> 2
- net Net-(IC1-CLKSEL0): track 0.00 -> 1.88 mm
- net Net-(IC1-CAP): track 1.01 -> 2.18 mm
- net Net-(IC1-ENV_SCL): track 0.00 -> 1.09 mm
- net Net-(IC1-PS0/WAKE): track 14.5 -> 15.5 mm
- net Net-(IC1-H_INTN): track 15.7 -> 15.4 mm, vias 0 -> 2
- net GND: vias 9 -> 10

Commit message: Logo added, doc updates, board tweaks, imgs
Parts:
- added G***: LOGO, LOGO, B.Cu at (151.7, 92.1)
Connections:
- C1 pad 2: /Bat+ -> vcc
- C2 pad 1: /Bat+ -> vcc
- PWR1 pad 1: /Bat+ -> vcc
- R2 pad 2: /Bat+ -> vcc
- U1 pad 15: /Bat+ -> vcc
Routing:
- net /Bat+: track 47.1 -> 21.2 mm
- net vcc: track 0.00 -> 25.8 mm
Other:
- board text added: "AZIMUTH"
- board text added: "V0.1"
- board text added: "WayWayWay"
