File: kicad/ESP32_BNO086/ESP32_BNO086.kicad_sch (KiCad schematic)
At the start: 14 parts, among them IC1 BNO086, U1 XIAO-ESP32-C3/S3

Commit message: wiring changes
Parts:
- removed RST/Center1: SW_Push, Button_Switch_SMD:SW_SPST_EVQP2_MiddlePushTravel_H2.5mm, symbol Switch:SW_Push
- added C4: 0.1uf, Capacitor_SMD:C_0402_1005Metric, symbol Device:C
- C3: value 0.1uf -> 10uf
Connections:
- net GND: now also C3.2, C4.2
- net at C3.1, IC1.5 (PS1), U1.12 (3V3): now also IC1.28 (VDDIO), IC1.3 (VDD), C4.1; no longer IC1.6 (PS0/WAKE)
- net at LS1.LOAD+: now also U1.7 (GPIO21_D6_TX); no longer U1.6 (GPIO7_D5_SCL)
- net at U1.5 (GPIO6_D4_SDA): now also IC1.14 (H_INTN)
- net at U1.3 (GPIO4_A2_D2): now also IC1.6 (PS0/WAKE); no longer IC1.18 (H_CSN)
- net at U1.4 (GPIO5_A3_D3): now also IC1.18 (H_CSN); no longer IC1.14 (H_INTN)
- net at FUNC1.2: now also U1.6 (GPIO7_D5_SCL); no longer U1.7 (GPIO21_D6_TX)
Other:
- moved on the sheet: C3, FUNC1

Commit message: Updated PCB design
Parts:
- added C5: 100nf, Capacitor_SMD:C_0402_1005Metric, symbol Device:C
- added R4: 10k, Resistor_SMD:R_0402_1005Metric, symbol Device:R
Connections:
- net GND: now also C5.1
- net at C3.1, C4.1, IC1.28 (VDDIO)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: now also R4.1
- net at IC1.4 (BOOTN): now also R4.2
- net at IC1.9 (CAP): now also C5.2
Other:
- moved on the sheet: C3

Commit message: pcb updates, doc updates, lib updates
Parts:
- removed FUNC1: SW_Push, Button_Switch_SMD:SW_SPST_EVQP2_MiddlePushTravel_H2.5mm, symbol Switch:SW_Push
- removed LS1: SMT-0540-T-9-R, 1_MyFootPrints:XDCR_SMT-0540-T-9-R, symbol 1_MyLib:SMT-0540-T-9-R
- removed S1: JS102011SAQN, 1_MyFootPrints:SW_JS102011SAQN, symbol 1_MyLib:JS102011SAQN
- added BUZZER1: MLT-5020, 1_MyFootPrints:BUZ-SMD_L5.0-W5.5-P4.60, symbol 1_MyLib:MLT-5020
- added FUNC1: HX 3X4X2-2P-1.6N TACTILE SWITCH, 1_MyFootPrints:KEY-SMD_L4.0-W3.0-LS4.9-1, symbol 1_MyLib:HX3X4X2-2P-1.6NTACTILESWITCH
- added PWR1: K3-1280S-K1, 1_MyFootPrints:SW-SMD_K3-1280S-K1, symbol 1_MyLib:K3-1280S-K1
- added R5, R6: 10k, Resistor_SMD:R_0402_1005Metric, symbol Device:R
- added R7, R8: 4.7k, Resistor_SMD:R_0402_1005Metric, symbol Device:R
- C1: LCSC Part (none) -> C19702; Manufacturer_Part_Number (none) -> CL10A106KP8NNNC
- C2: LCSC Part (none) -> C14663; Manufacturer_Part_Number (none) -> CC0603KRX7R9BB104
- C3: footprint Capacitor_SMD:C_0402_1005Metric -> Capacitor_SMD:C_0603_1608Metric; LCSC Part (none) -> C19702; Manufacturer_Part_Number (none) -> CL10A106KP8NNNC
- C4: footprint Capacitor_SMD:C_0402_1005Metric -> Capacitor_SMD:C_0603_1608Metric; LCSC Part (none) -> C14663; Manufacturer_Part_Number (none) -> CC0603KRX7R9BB104
- C5: LCSC Part (none) -> C77020; Manufacturer_Part_Number (none) -> GRM155R71H104KE14D
- IC1: Manufacturer_Name BOSCH -> BOSCH / CEVA Technologies, Inc.; Mouser Part Number (none) -> 526-BNO086
- LED1: LCSC Part (none) -> C21260817; Manufacturer_Part_Number (none) -> YLED0402R
- PH2.0: value Conn_01x02_Socket -> S2B-PH-SM4-TB(LF)(SN); LCSC Part (none) -> C295747; Manufacturer_Part_Number (none) -> S2B-PH-SM4-TB(LF)(SN)
- R1, R2: LCSC Part (none) -> C2907013; Manufacturer_Part_Number (none) -> FRC0603F2203TS
- R3: LCSC Part (none) -> C114877; Manufacturer_Part_Number (none) -> RC0402FR-07470RL
- R4: LCSC Part (none) -> C60490; Manufacturer_Part_Number (none) -> RC0402FR-0710KL
- U1: value XIAO-ESP32-C3/S3 -> XIAO-ESP32-C3; Manufacturer_Name (none) -> SEEED STUDIO; Manufacturer_Part_Number (none) -> 113991054; Mouser Part Number (none) -> 713-113991054
Connections:
- net Bat+: now also PWR1.1, PWR1.2
- net GND: now also C3.1, C4.1, BUZZER1.2 (-), FUNC1.2; no longer C3.2, C4.2
- net at IC1.28 (VDDIO), IC1.3 (VDD), IC1.5 (PS1)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: now also C3.2, C4.2, R5.1, R6.1, R7.1, R8.1; no longer C3.1, C4.1
- net at U1.7 (GPIO21_D6_TX): now also BUZZER1.1 (+)
- net at IC1.6 (PS0/WAKE), U1.3 (GPIO4_A2_D2): now also R5.2
- net at U1.6 (GPIO7_D5_SCL): now also FUNC1.1
- net at IC1.10 (CLKSEL0): now also R6.2
- net at IC1.15 (ENV_SCL): now also R7.2
- net at IC1.16 (ENV_SDA): now also R8.2
Other:
- moved on the sheet: C5
